File: hardware/glm5va/glm5va.kicad_sch (KiCad schematic)
At the start: 21 parts, among them J1 Conn_02x10_Odd_Even, J2 JIN, J3 POWER, U1 74HC245, U2 74HC245

Commit message: adding pdf for schematic
Other:
- title: (none) -> Convert 2.5V signals -> 5V
Changed lines of the file:
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@@
 	(generator_version "8.0")
 	(paper "A4")
+	(title_block
+		(title "Convert 2.5V signals -> 5V")
+		(date "2025-01-20")
+		(rev "v0.1")
+	)
 	(junction
 		(at 252.73 24.13)
